Commit message: Co-authored-by: SHASHANK H S <Shashankhs17@users.noreply.github.com>

File: env-setup/humanoid.urdf (robot description, URDF)
Before this commit: robot dumpUrdf, 16 links, 15 joints
Joints:
- joint right_hip: axis 0.000000 0.000000 1.000000 -> (none); limit lower=-1.57 upper=1.57 effort=1000.0 velocity=0.5 -> (none); type revolute -> fixed

Commit message: new branch created

File: env-setup/humanoid.urdf (robot description, URDF)
Before this commit: robot dumpUrdf, 16 links, 15 joints
Joints:
- joint right_hip: axis (none) -> 0.000000 0.000000 1.000000; limit (none) -> lower=-1.57 upper=1.57 effort=1000.0 velocity=0.5; type fixed -> revolute

Commit message: trial to find out the optimum time step value

File: env-setup/humanoid.urdf (robot description, URDF)
Before this commit: robot dumpUrdf, 16 links, 15 joints
Joints:
- joint right_ankle: axis 0.000000 0.000000 1.000000 -> (none); limit lower=-0.785 upper=0. effort=1000.0 velocity=0.5 -> (none); type revolute -> fixed
- joint right_knee: limit lower=-3.14 upper=0. effort=1000.0 velocity=0.5 -> lower=-3.14 upper=0. effort=0 velocity=200
